Commit message: add jaka_ros2

File: src/tracer_jaka_moveit_config/config/tracer_jaka_zu5.ros2_control.xacro (robot description, xacro)
@@ -14,4 +14,5 @@
                 </state_interface>
                 <state_interface name="velocity"/>
+                <state_interface name="effort"/>
             </joint>
             <joint name="joint_2">
@@ -21,4 +22,5 @@
                 </state_interface>
                 <state_interface name="velocity"/>
+                <state_interface name="effort"/>
             </joint>
             <joint name="joint_3">
@@ -28,4 +30,5 @@
                 </state_interface>
                 <state_interface name="velocity"/>
+                <state_interface name="effort"/>
             </joint>
             <joint name="joint_4">
@@ -35,4 +38,5 @@
                 </state_interface>
                 <state_interface name="velocity"/>
+                <state_interface name="effort"/>
             </joint>
             <joint name="joint_5">
@@ -42,4 +46,5 @@
                 </state_interface>
                 <state_interface name="velocity"/>
+                <state_interface name="effort"/>
             </joint>
             <joint name="joint_6">
@@ -49,11 +54,5 @@
                 </state_interface>
                 <state_interface name="velocity"/>
-            </joint>
-            <joint name="gripper_finger1_joint">
-                <command_interface name="position"/>
-                <state_interface name="position">
-                  <param name="initial_value">${initial_positions['gripper_finger1_joint']}</param>
-                </state_interface>
-                <state_interface name="velocity"/>
+                <state_interface name="effort"/>
             </joint>
         </ros2_control>
