Commit message: add jaka_tcp_sensor

File: src/jaka_ros2/src/jaka_description/urdf/tracer_jaka_zu5.urdf (robot description, URDF)
Before this commit: robot tracer_jaka_zu5, 42 links, 41 joints
Joints:
- joint gripper_finger1_finger_joint: type continuous -> fixed
- joint gripper_finger1_finger_tip_joint: type continuous -> fixed
- joint gripper_finger1_inner_knuckle_joint: type continuous -> fixed
- joint gripper_finger1_joint: type revolute -> fixed
- joint gripper_finger2_finger_joint: type continuous -> fixed
- joint gripper_finger2_finger_tip_joint: type continuous -> fixed
- joint gripper_finger2_inner_knuckle_joint: type continuous -> fixed
- joint gripper_finger2_joint: type revolute -> fixed

Commit message: revise tcp_link

File: src/jaka_ros2/src/jaka_description/urdf/tracer_jaka_zu5.urdf (robot description, URDF)
Before this commit: robot tracer_jaka_zu5, 42 links, 41 joints
Joints:
- joint gripper_base_joint: origin xyz=0 0 0.036 rpy=0 0 0 -> xyz=0 0 0.005 rpy=0 0 -0.7853
- joint jk_se_vi_200_joint: origin xyz=0 0 0  rpy=0 0 0 -> xyz=0 0 0.0315  rpy=0 0 0.785398

File: src/tracer_jaka_moveit_config/config/tracer_jaka_zu5.ros2_control.xacro (robot description, xacro)
@@ -6,6 +6,6 @@
             <hardware>
                 <!-- By default, set up controllers for simulation. This won't work on real hardware -->
-                <!-- <plugin>mock_components/GenericSystem</plugin> -->
-                <plugin>jaka_hardware_interface/JakaHardwareInterface</plugin>
+                <plugin>mock_components/GenericSystem</plugin>
+                <!-- <plugin>jaka_hardware_interface/JakaHardwareInterface</plugin> -->
                 <param name="robot_ip">10.5.5.100</param>
                 <param name="local_ip">10.5.5.127</param>

Commit message: 添加重力补偿

File: src/jaka_ros2/src/jaka_description/urdf/tracer_jaka_zu5.urdf (robot description, URDF)
Before this commit: robot tracer_jaka_zu5, 42 links, 41 joints
Joints:
- joint base_to_jaka: origin xyz=0 0 0.218 rpy=0 0 0 -> xyz=0 0 0.221 rpy=-0.02 0 0

File: src/tracer_jaka_moveit_config/config/tracer_jaka_zu5.ros2_control.xacro (robot description, xacro)
@@ -6,6 +6,6 @@
             <hardware>
                 <!-- By default, set up controllers for simulation. This won't work on real hardware -->
-                <plugin>mock_components/GenericSystem</plugin>
-                <!-- <plugin>jaka_hardware_interface/JakaHardwareInterface</plugin> -->
+                <!-- <plugin>mock_components/GenericSystem</plugin> -->
+                <plugin>jaka_hardware_interface/JakaHardwareInterface</plugin>
                 <param name="robot_ip">10.5.5.100</param>
                 <param name="local_ip">10.5.5.127</param>
@@ -17,5 +17,4 @@
                 </state_interface>
                 <state_interface name="velocity"/>
-                <state_interface name="effort"/>
             </joint>
             <joint name="joint_2">
@@ -25,5 +24,4 @@
                 </state_interface>
                 <state_interface name="velocity"/>
-                <state_interface name="effort"/>
             </joint>
             <joint name="joint_3">
@@ -33,5 +31,4 @@
                 </state_interface>
                 <state_interface name="velocity"/>
-                <state_interface name="effort"/>
             </joint>
             <joint name="joint_4">
@@ -41,5 +38,4 @@
                 </state_interface>
                 <state_interface name="velocity"/>
-                <state_interface name="effort"/>
             </joint>
             <joint name="joint_5">
@@ -49,5 +45,4 @@
                 </state_interface>
                 <state_interface name="velocity"/>
-                <state_interface name="effort"/>
             </joint>
             <joint name="joint_6">
@@ -57,5 +52,4 @@
                 </state_interface>
                 <state_interface name="velocity"/>
-                <state_interface name="effort"/>
             </joint>
             <sensor name="tcp_fts_sensor">

File: src/tracer_jaka_moveit_config/config/tracer_jaka_zu5.urdf.xacro (robot description, xacro)
@@ -6,4 +6,4 @@
     <!-- Import control_xacro -->
     <xacro:include filename="tracer_jaka_zu5.ros2_control.xacro" />
-    <xacro:tracer_jaka_zu5_ros2_control name="FakeSystem" initial_positions_file="$(arg initial_positions_file)"/>
+    <xacro:tracer_jaka_zu5_ros2_control name="RealSystem" initial_positions_file="$(arg initial_positions_file)"/>
 </robot>

Commit message: finish JTC chained control

File: src/jaka_ros2/src/jaka_description/urdf/tracer_jaka_zu5.urdf (robot description, URDF)
Before this commit: robot tracer_jaka_zu5, 42 links, 41 joints
Joints:
- joint gripper_center_joint: origin xyz=0 0 0.22  rpy=0 0 0 -> xyz=0 0 0.1885  rpy=0 0 -0.785398; parent Link_6_45 -> jk_se_vi_200_link

Commit message: changed tcp compensate from node to hardware

File: src/jaka_ros2/src/jaka_description/urdf/tracer_jaka_zu5.urdf (robot description, URDF)
Before this commit: robot tracer_jaka_zu5, 42 links, 41 joints
Joints:
- joint gripper_center_joint: origin xyz=0 0 0.1885  rpy=0 0 -0.785398 -> xyz=0 0 0.205  rpy=0 0 -0.785398

File: src/tracer_jaka_moveit_config/config/tracer_jaka_zu5.ros2_control.xacro (robot description, xacro)
@@ -10,4 +10,8 @@
                 <param name="robot_ip">10.5.5.100</param>
                 <param name="local_ip">10.5.5.127</param>
+                <param name="sensor_to_tcp_offset_x">0.0</param>
+                <param name="sensor_to_tcp_offset_y">0.0</param>
+                <param name="sensor_to_tcp_offset_z">0.205</param>
+                <param name="sensor_z_angle">0.785398</param>
             </hardware>
             <joint name="joint_1">

Commit message: add path tracker

File: src/jaka_ros2/src/jaka_description/urdf/tracer_jaka_zu5.urdf (robot description, URDF)
Before this commit: robot tracer_jaka_zu5, 42 links, 41 joints
Links:
- added link world
Joints:
- added joint world_to_base_link=: type fixed, parent world, child base_link, origin xyz=0 0 0.136 rpy=0 0 0

File: src/tracer_jaka_moveit_config/config/tracer_jaka_zu5.ros2_control.xacro (robot description, xacro)
@@ -6,6 +6,6 @@
             <hardware>
                 <!-- By default, set up controllers for simulation. This won't work on real hardware -->
-                <!-- <plugin>mock_components/GenericSystem</plugin> -->
-                <plugin>jaka_hardware_interface/JakaHardwareInterface</plugin>
+                <plugin>mock_components/GenericSystem</plugin>
+                <!-- <plugin>jaka_hardware_interface/JakaHardwareInterface</plugin> -->
                 <param name="robot_ip">10.5.5.100</param>
                 <param name="local_ip">10.5.5.127</param>

Commit message: combine path with force

File: src/jaka_ros2/src/jaka_description/urdf/tracer_jaka_zu5.urdf (robot description, URDF)
Before this commit: robot tracer_jaka_zu5, 43 links, 42 joints
Joints:
- joint gripper_center_joint: origin xyz=0 0 0.205  rpy=0 0 -0.785398 -> xyz=0 -0.025 0.225  rpy=0.5235 0 -0.785398

Commit message: add sheep cloud process

File: src/jaka_ros2/src/jaka_description/urdf/tracer_jaka_zu5.urdf (robot description, URDF)
Before this commit: robot tracer_jaka_zu5, 43 links, 42 joints
Links:
- removed link gripper_base_link
- removed link gripper_center_link
- removed link gripper_finger1_finger_link
- removed link gripper_finger1_finger_tip_link
- removed link gripper_finger1_inner_knuckle_link
- removed link gripper_finger1_knuckle_link
- removed link gripper_finger2_finger_link
- removed link gripper_finger2_finger_tip_link
- removed link gripper_finger2_inner_knuckle_link
- removed link gripper_finger2_knuckle_link
- added link shaver_link; collision mesh filename=package://jaka_description/meshes/shaver/shaver.stl scale=0.001 0.001 0.001; visual mesh filename=package://jaka_description/meshes/shaver/shaver.stl scale=0.001 0.001 0.001
- added link tool0
Joints:
- removed joint gripper_base_joint
- removed joint gripper_center_joint
- removed joint gripper_finger1_finger_joint
- removed joint gripper_finger1_finger_tip_joint
- removed joint gripper_finger1_inner_knuckle_joint
- removed joint gripper_finger1_joint
- removed joint gripper_finger2_finger_joint
- removed joint gripper_finger2_finger_tip_joint
- removed joint gripper_finger2_inner_knuckle_joint
- removed joint gripper_finger2_joint
- added joint shaver_joint: type fixed, parent jk_se_vi_200_link, child shaver_link, origin xyz=-0.01768 -0.01768 0.005 rpy=0 0 -0.785398
- added joint tool0_joint: type fixed, parent shaver_link, child tool0, origin xyz=0 -0.005 0.225 rpy=0.3491 0 0
- joint connector_base_joint: origin xyz=0 -0.0365 -0.005 rpy=3.14 -1.57 -1.57 -> xyz=-0.0315 -0.0315 0 rpy=0 -1.57 0.78; parent gripper_base_link -> jk_se_vi_200_link

File: src/tracer_jaka_moveit_config/config/tracer_jaka_zu5.ros2_control.xacro (robot description, xacro)
@@ -6,12 +6,23 @@
             <hardware>
                 <!-- By default, set up controllers for simulation. This won't work on real hardware -->
-                <!-- <plugin>mock_components/GenericSystem</plugin> -->
-                <plugin>jaka_hardware_interface/JakaHardwareInterface</plugin>
+                <plugin>mock_components/GenericSystem</plugin>
+                <!-- <plugin>jaka_hardware_interface/JakaHardwareInterface</plugin> -->
                 <param name="robot_ip">10.5.5.100</param>
                 <param name="local_ip">10.5.5.127</param>
-                <param name="sensor_to_tcp_offset_x">0.0</param>
-                <param name="sensor_to_tcp_offset_y">0.0</param>
-                <param name="sensor_to_tcp_offset_z">0.205</param>
-                <param name="sensor_z_angle">0.785398</param>
+                <!-- 力传感器偏置 -->
+                <param name="ft_bias_fx">-9.80</param>
+                <param name="ft_bias_fy">-6.78</param>
+                <param name="ft_bias_fz">-6.00</param>
+                <param name="ft_bias_tx">0.54</param>
+                <param name="ft_bias_ty">-0.63</param>
+                <param name="ft_bias_tz">0.03</param>
+                <param name="r_t_s_x">0.0</param>
+                <param name="r_t_s_y">-0.05</param>
+                <param name="r_t_s_z">-0.226</param>
+                <!-- 死区 -->
+                <param name="ft_deadband_force">1.0</param>
+                <param name="ft_deadband_torque">0.00</param>
+                <!-- 滤波系数 -->
+                <param name="ft_filter_alpha">0.1</param>
             </hardware>
             <joint name="joint_1">

File: src/tracer_jaka_moveit_config/config/tracer_jaka_zu5.urdf.xacro (robot description, xacro)
@@ -6,4 +6,4 @@
     <!-- Import control_xacro -->
     <xacro:include filename="tracer_jaka_zu5.ros2_control.xacro" />
-    <xacro:tracer_jaka_zu5_ros2_control name="RealSystem" initial_positions_file="$(arg initial_positions_file)"/>
+    <xacro:tracer_jaka_zu5_ros2_control name="FakeSystem" initial_positions_file="$(arg initial_positions_file)"/>
 </robot>

Commit message: pick and place demo

File: src/jaka_ros2/src/jaka_description/urdf/tracer_jaka_zu5.urdf (robot description, URDF)
Before this commit: robot tracer_jaka_zu5, 35 links, 34 joints
Links:
- removed link shaver_link
- removed link tool0
- added link gripper_base_link, mass 0.83416; collision mesh filename=package://jaka_description/meshes/dh_robotics_ag95_descript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 scale=0.001 0.001 0.001; visual mesh filename=package://jaka_description/meshes/dh_robotics_ag95_descript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 scale=0.001 0.001 0.001
- added link gripper_center_link
- added link gripper_finger1_finger_link, mass 0.0222871; collision mesh filename=package://jaka_description/meshes/dh_robotics_ag95_descript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 scale=0.001 0.001 0.001; visual mesh filename=package://jaka_description/meshes/dh_robotics_ag95_descript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 scale=0.001 0.001 0.001
- added link gripper_finger1_finger_tip_link, mass 0.0124305; collision mesh filename=package://jaka_description/meshes/dh_robotics_ag95_descript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 scale=0.001 0.001 0.001; visual mesh filename=package://jaka_description/meshes/dh_robotics_ag95_descript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 scale=0.001 0.001 0.001
- added link gripper_finger1_inner_knuckle_link, mass 0.0318004; collision mesh filename=package://jaka_description/meshes/dh_robotics_ag95_descript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 scale=0.001 0.001 0.001; visual mesh filename=package://jaka_description/meshes/dh_robotics_ag95_descript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 scale=0.001 0.001 0.001
- added link gripper_finger1_knuckle_link, mass 0.011111; collision mesh filename=package://jaka_description/meshes/dh_robotics_ag95_descript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 scale=0.001 0.001 0.001; visual mesh filename=package://jaka_description/meshes/dh_robotics_ag95_descript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 scale=0.001 0.001 0.001
- added link gripper_finger2_finger_link, mass 0.0222871; collision mesh filename=package://jaka_description/meshes/dh_robotics_ag95_descript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 scale=0.001 0.001 0.001; visual mesh filename=package://jaka_description/meshes/dh_robotics_ag95_descript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 scale=0.001 0.001 0.001
- added link gripper_finger2_finger_tip_link, mass 0.0124305; collision mesh filename=package://jaka_description/meshes/dh_robotics_ag95_descript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 scale=0.001 0.001 0.001; visual mesh filename=package://jaka_description/meshes/dh_robotics_ag95_descript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 scale=0.001 0.001 0.001
- added link gripper_finger2_inner_knuckle_link, mass 0.0318004; collision mesh filename=package://jaka_description/meshes/dh_robotics_ag95_descript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 scale=0.001 0.001 0.001; visual mesh filename=package://jaka_description/meshes/dh_robotics_ag95_descript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 scale=0.001 0.001 0.001
- added link gripper_finger2_knuckle_link, mass 0.011111; collision mesh filename=package://jaka_description/meshes/dh_robotics_ag95_descript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 scale=0.001 0.001 0.001; visual mesh filename=package://jaka_description/meshes/dh_robotics_ag95_descript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 scale=0.001 0.001 0.001
Joints:
- removed joint shaver_joint
- removed joint tool0_joint
- added joint gripper_base_joint: type fixed, parent jk_se_vi_200_link, child gripper_base_link, origin xyz=0 0 0.005 rpy=0 0 -0.7853
- added joint gripper_center_joint: type fixed, parent jk_se_vi_200_link, child gripper_center_link, origin xyz=0 0 0.225  rpy=0 0 -0.785398
- added joint gripper_finger1_finger_joint: type continuous, parent gripper_finger1_knuckle_link, child gripper_finger1_finger_link, origin xyz=0.0292080077784 0.0 -0.0227132622407 rpy=0 0 0, axis 0 -1 0, limit lower=-3.14 upper=3.14 effort=0.1 velocity=100.0, mimic joint=gripper_finger1_joint multiplier=0.4563942 offset=0
- added joint gripper_finger1_finger_tip_joint: type continuous, parent gripper_finger1_inner_knuckle_link, child gripper_finger1_finger_tip_link, origin xyz=0.0394969463769 0.0 0.0382752038125  rpy=0.0 0.0 0.0, axis 0 1 0, limit lower=-3.14 upper=3.14 effort=0.1 velocity=100.0, mimic joint=gripper_finger1_joint multiplier=1.49462955
- added joint gripper_finger1_inner_knuckle_joint: type continuous, parent gripper_base_link, child gripper_finger1_inner_knuckle_link, origin xyz=-0.016 0 0.10586 rpy=0.0 0.0 3.141592653589793, axis 0 -1 0, limit lower=-3.14 upper=3.14 effort=0.1 velocity=100.0, mimic joint=gripper_finger1_joint multiplier=1.49462955 offset=0
- added joint gripper_finger1_joint: type revolute, parent gripper_base_link, child gripper_finger1_knuckle_link, origin xyz=-0.016 0 0.10586 rpy=0.0 0.0 3.141592653589793, axis 0 -1 0, limit lower=0.0 upper=0.65 effort=1000 velocity=2.0
- added joint gripper_finger2_finger_joint: type continuous, parent gripper_finger2_knuckle_link, child gripper_finger2_finger_link, origin xyz=0.0292080077784 0.0 -0.0227132622407 rpy=0 0 0, axis 0 -1 0, limit lower=-3.14 upper=3.14 effort=0.1 velocity=100.0, mimic joint=gripper_finger1_joint multiplier=0.4563942 offset=0
- added joint gripper_finger2_finger_tip_joint: type continuous, parent gripper_finger2_inner_knuckle_link, child gripper_finger2_finger_tip_link, origin xyz=0.0394969463769  0.0 0.0382752038125   rpy=0.0 0.0 0.0, axis 0 1 0, limit lower=-3.14 upper=3.14 effort=0.1 velocity=100.0, mimic joint=gripper_finger1_joint multiplier=1.49462955
- added joint gripper_finger2_inner_knuckle_joint: type continuous, parent gripper_base_link, child gripper_finger2_inner_knuckle_link, origin xyz=0.016 0 0.10586 rpy=0.0 0.0 0.0, axis 0 -1 0, limit lower=-3.14 upper=3.14 effort=0.1 velocity=100.0, mimic joint=gripper_finger1_joint multiplier=1.49462955 offset=0
- added joint gripper_finger2_joint: type revolute, parent gripper_base_link, child gripper_finger2_knuckle_link, origin xyz=0.016  0 0.10586  rpy=0.0 0.0 0.0, axis 0 -1 0, limit lower=-3.14 upper=3.14 effort=1000 velocity=100.0, mimic joint=gripper_finger1_joint

Commit message: almost finish polish

File: src/jaka_ros2/src/jaka_description/urdf/tracer_jaka_zu5.urdf (robot description, URDF)
Before this commit: robot tracer_jaka_zu5, 43 links, 42 joints
Joints:
- joint gripper_center_joint: origin xyz=0 0 0.225  rpy=0 0 -0.785398 -> xyz=0 0 0.27  rpy=0 0 -0.785398

File: src/tracer_jaka_moveit_config/config/tracer_jaka_zu5.ros2_control.xacro (robot description, xacro)
@@ -9,20 +9,20 @@
                 <!-- <plugin>mock_components/GenericSystem</plugin> -->
                 <param name="robot_ip">10.5.5.100</param>
-                <param name="local_ip">10.5.5.166</param>
+                <param name="local_ip">10.5.5.127</param>
                 <!-- 力传感器偏置 -->
-                <param name="ft_bias_fx">-9.80</param>
-                <param name="ft_bias_fy">-6.78</param>
-                <param name="ft_bias_fz">-6.00</param>
-                <param name="ft_bias_tx">0.54</param>
-                <param name="ft_bias_ty">-0.63</param>
-                <param name="ft_bias_tz">0.03</param>
-                <param name="r_t_s_x">0.0</param>
-                <param name="r_t_s_y">-0.05</param>
-                <param name="r_t_s_z">-0.226</param>
+                <param name="ft_bias_fx">-7.79</param>
+                <param name="ft_bias_fy">-7.63</param>
+                <param name="ft_bias_fz">-0.21</param>
+                <param name="ft_bias_tx">0.74</param>
+                <param name="ft_bias_ty">-0.73</param>
+                <param name="ft_bias_tz">-0.02</param>
+                <param name="r_t_s_x">-0.0080</param>
+                <param name="r_t_s_y">-0.0157</param>
+                <param name="r_t_s_z">0.27</param>
                 <!-- 死区 -->
-                <param name="ft_deadband_force">1.0</param>
+                <param name="ft_deadband_force">0.5</param>
                 <param name="ft_deadband_torque">0.00</param>
                 <!-- 滤波系数 -->
-                <param name="ft_filter_alpha">0.1</param>
+                <param name="ft_filter_alpha">0.0</param>
             </hardware>
             <joint name="joint_1">
